Commit message: 動く状態に更新

File: kuams3_description/urdf/kuams3.xacro (robot description, xacro)
@@ -132,10 +132,19 @@
   <axis xyz="-1.0 0.0 0.0"/>
 </joint>
+<link name="front_sensor_link">
+</link>
+<joint name="livox_front_sensor_joint" type="fixed">
+    <!-- <origin rpy="0 0 1.57" xyz="0 0.18 0.45"/> -->
+    <origin rpy="0 0 1.57" xyz="0 0.18 0.45"/>
+    <parent link="base_link"/>
+    <child link="front_sensor_link"/>
+</joint>
 <!-- laser -->
 <link name="livox_frame">
 </link>
 <joint name="laser_joint" type="fixed">
-    <origin rpy="0 0 0" xyz="0 -0.1 0.18"/>
-    <parent link="base_link"/>
+    <!-- <origin rpy="0 0.785 0" xyz="0 0 0"/> -->
+    <origin rpy="0 0 0" xyz="0 0 0"/>
+    <parent link="front_sensor_link"/>
     <child link="livox_frame"/>
 </joint>

Commit message: nav2で動く状態に更新

File: kuams3_description/urdf/kuams3.xacro (robot description, xacro)
@@ -6,5 +6,5 @@
   <parent link="base_footprint"/>
   <child link="base_link" />
-  <origin xyz="0 0 0" rpy="0 0 ${radians(-90)}"/>
+  <origin xyz="0 0 0" rpy="0 0 0"/>
 </joint>
 <link name="base_link">
@@ -15,5 +15,5 @@
   </inertial>
   <visual>
-    <origin xyz="0 0 0" rpy="0 0 0"/>
+    <origin xyz="0 0 0" rpy="0 0 ${radians(-90)}"/>
     <geometry>
       <mesh filename="package://kuams3_description/meshes/base_link.stl" scale="0.001 0.001 0.001"/>
@@ -22,5 +22,5 @@
   </visual>
   <collision>
-    <origin xyz="0 0 0" rpy="0 0 0"/>
+    <origin xyz="0 0 0" rpy="0 0 ${radians(-90)}"/>
     <geometry>
       <mesh filename="package://kuams3_description/meshes/base_link.stl" scale="0.001 0.001 0.001"/>
@@ -35,5 +35,5 @@
   </inertial>
   <visual>
-    <origin xyz="0.0875 -0.12 -0.076" rpy="0 0 0"/>
+    <origin xyz="-0.12 -0.0875 -0.076" rpy="0 0 ${radians(-90)}"/>
     <geometry>
       <mesh filename="package://kuams3_description/meshes/front_left_wheel_1.stl" scale="0.001 0.001 0.001"/>
@@ -42,5 +42,5 @@
   </visual>
   <collision>
-    <origin xyz="0.0875 -0.12 -0.076" rpy="0 0 0"/>
+    <origin xyz="-0.12 -0.0875 -0.076" rpy="0 0 ${radians(-90)}"/>
     <geometry>
       <mesh filename="package://kuams3_description/meshes/front_left_wheel_1.stl" scale="0.001 0.001 0.001"/>
@@ -55,5 +55,5 @@
   </inertial>
   <visual>
-    <origin xyz="-0.0875 -0.12 -0.076" rpy="0 0 0"/>
+    <origin xyz="-0.12 0.0875 -0.076" rpy="0 0 ${radians(-90)}"/>
     <geometry>
       <mesh filename="package://kuams3_description/meshes/front_right_wheel_1.stl" scale="0.001 0.001 0.001"/>
@@ -62,5 +62,5 @@
   </visual>
   <collision>
-    <origin xyz="-0.0875 -0.12 -0.076" rpy="0 0 0"/>
+    <origin xyz="-0.12 0.0875 -0.076" rpy="0 0 ${radians(-90)}"/>
     <geometry>
       <mesh filename="package://kuams3_description/meshes/front_right_wheel_1.stl" scale="0.001 0.001 0.001"/>
@@ -75,5 +75,5 @@
   </inertial>
   <visual>
-    <origin xyz="-0.0875 0.12 -0.076" rpy="0 0 0"/>
+    <origin xyz="0.12 0.0875 -0.076" rpy="0 0 ${radians(-90)}"/>
     <geometry>
       <mesh filename="package://kuams3_description/meshes/back_right_wheel_1.stl" scale="0.001 0.001 0.001"/>
@@ -82,5 +82,5 @@
   </visual>
   <collision>
-    <origin xyz="-0.0875 0.12 -0.076" rpy="0 0 0"/>
+    <origin xyz="0.12 0.0875 -0.076" rpy="0 0 ${radians(-90)}"/>
     <geometry>
       <mesh filename="package://kuams3_description/meshes/back_right_wheel_1.stl" scale="0.001 0.001 0.001"/>
@@ -95,5 +95,5 @@
   </inertial>
   <visual>
-    <origin xyz="0.0875 0.12 -0.076" rpy="0 0 0"/>
+    <origin xyz="0.12 -0.0875 -0.076" rpy="0 0 ${radians(-90)}"/>
     <geometry>
       <mesh filename="package://kuams3_description/meshes/back_left_wheel_1.stl" scale="0.001 0.001 0.001"/>
@@ -102,5 +102,5 @@
   </visual>
   <collision>
-    <origin xyz="0.0875 0.12 -0.076" rpy="0 0 0"/>
+    <origin xyz="0.12 -0.0875 -0.076" rpy="0 0 ${radians(-90)}"/>
     <geometry>
       <mesh filename="package://kuams3_description/meshes/back_left_wheel_1.stl" scale="0.001 0.001 0.001"/>
@@ -109,11 +109,11 @@
 </link>
 <joint name="front_left_joint" type="continuous">
-  <origin xyz="-0.0875 0.12 0.076" rpy="0 0 0"/>
+  <origin xyz="0.12 0.0875 0.076" rpy="0 0 0"/>
   <parent link="base_link"/>
   <child link="front_left_wheel_1"/>
-  <axis xyz="-1.0 0.0 0.0"/>
+  <axis xyz="0.0 -1.0 0.0"/>
 </joint>
 <joint name="front_right_joint" type="continuous">
-  <origin xyz="0.0875 0.12 0.076" rpy="0 0 0"/>
+  <origin xyz="0.12 -0.0875 0.076" rpy="0 0 0"/>
   <parent link="base_link"/>
   <child link="front_right_wheel_1"/>
@@ -121,5 +121,5 @@
 </joint>
 <joint name="back_right_joint" type="continuous">
-  <origin xyz="0.0875 -0.12 0.076" rpy="0 0 0"/>
+  <origin xyz="-0.12 -0.0875 0.076" rpy="0 0 0"/>
   <parent link="base_link"/>
   <child link="back_right_wheel_1"/>
@@ -127,5 +127,5 @@
 </joint>
 <joint name="back_left_joint" type="continuous">
-  <origin xyz="-0.0875 -0.12 0.076" rpy="0 0 0"/>
+  <origin xyz="-0.12 0.0875 0.076" rpy="0 0 0"/>
   <parent link="base_link"/>
   <child link="back_left_wheel_1"/>
@@ -136,5 +136,5 @@
 <joint name="livox_front_sensor_joint" type="fixed">
     <!-- <origin rpy="0 0 1.57" xyz="0 0.18 0.45"/> -->
-    <origin rpy="0 0 1.57" xyz="0 0.18 0.45"/>
+    <origin rpy="0 0 0" xyz="0.18 0 0.45"/>
     <parent link="base_link"/>
     <child link="front_sensor_link"/>
